Commit message: feat: complete sensor integration, multi-radar, systemd deploy, map versioning

File: src/wheelchair_description/urdf/wheelchair.urdf.xacro (robot description, xacro)
@@ -78,4 +78,32 @@
     <origin xyz="0.45 0.0 0.65" rpy="0.0 -0.0873 0.0"/>
   </joint>
+  <link name="xtm60_left_link">
+    <visual>
+      <origin xyz="0 0 0" rpy="0 0 0"/>
+      <geometry>
+        <box size="0.10 0.06 0.04"/>
+      </geometry>
+      <material name="laser_red"/>
+    </visual>
+  </link>
+  <joint name="xtm60_left_fixed_joint" type="fixed">
+    <parent link="base_link"/>
+    <child link="xtm60_left_link"/>
+    <origin xyz="0.45 0.24 0.65" rpy="0.0 -0.0873 0.0"/>
+  </joint>
+  <link name="xtm60_right_link">
+    <visual>
+      <origin xyz="0 0 0" rpy="0 0 0"/>
+      <geometry>
+        <box size="0.10 0.06 0.04"/>
+      </geometry>
+      <material name="laser_red"/>
+    </visual>
+  </link>
+  <joint name="xtm60_right_fixed_joint" type="fixed">
+    <parent link="base_link"/>
+    <child link="xtm60_right_link"/>
+    <origin xyz="0.45 -0.24 0.65" rpy="0.0 -0.0873 0.0"/>
+  </joint>
   <link name="imu_link">
     <visual>

Commit message: Camera calibration, dual-cam colorizer, XT-M60 optical frame + diagnostics
- camera_adapter: publish camera_info from calibration YAML; MJPG fourcc;
  per-camera 180deg rotation for upside-down mounts
- rgb_cloud_colorizer: optional aux camera (color main first, fill from aux);
  approximate forward-camera extrinsics (no calibration required to start)
- calib/: left/right intrinsics (+unrotated backups), printable checkerboard
- scripts: solve_cam_lidar_extrinsic (PnP), pick_image_points, log_clicked_points
- XT-M60 link set to OPTICAL frame (z-forward) so points map into base_link;
  fusion per-stage diagnostic logging
- bringup_3d_slam: graceful skip if topic_tools missing; wire aux camera
- docs/calibration_checklist: full intrinsic+extrinsic command guide

File: src/wheelchair_description/urdf/wheelchair.urdf.xacro (robot description, xacro)
@@ -90,5 +90,8 @@
     <parent link="base_link"/>
     <child link="xtm60_left_link"/>
-    <origin xyz="0.45 0.24 0.65" rpy="0.0 -0.0873 0.0"/>
+    <!-- XT-M60 (ToF camera) publishes points in OPTICAL convention (z forward,
+         x right, y down). This rpy makes the link an optical frame so optical-z
+         maps to base_link +x (forward). -->
+    <origin xyz="0.45 0.24 0.65" rpy="-1.5708 0.0 -1.5708"/>
   </joint>
   <link name="xtm60_right_link">
@@ -104,5 +107,6 @@
     <parent link="base_link"/>
     <child link="xtm60_right_link"/>
-    <origin xyz="0.45 -0.24 0.65" rpy="0.0 -0.0873 0.0"/>
+    <!-- optical frame: z forward -> base_link +x (see left joint note) -->
+    <origin xyz="0.45 -0.24 0.65" rpy="-1.5708 0.0 -1.5708"/>
   </joint>
   <link name="imu_link">

Commit message: feat: 新增XT-M60实时PointCloud+Amp显示工具，优化建图配置
- 新增experiments/amp_view全套工具，包含Python处理节点、启动脚本、RViz配置与使用文档，可实时复刻上位机的PointCloud+Amp显示效果，无需启动建图和电机
- 调整双雷达融合配置的点云高度裁剪范围，适配硬件安装高度，过滤无效的地板与天花板点云
- 修正轮椅URDF中XT-M60的安装高度：左侧雷达调整为实际0.45m，右侧雷达标注占位并提示需校准
- 优化RTAB-Map建图参数：启用法线分割区分地面与障碍物，解决广角雷达误识别地板为障碍物导致2D地图全黑的问题；调整网格最大有效范围为8m，改进参数传递方式确保配置生效
- 在手动建图RViz配置中新增右侧XT-M60点云的显示项

File: src/wheelchair_description/urdf/wheelchair.urdf.xacro (robot description, xacro)
@@ -92,6 +92,9 @@
     <!-- XT-M60 (ToF camera) publishes points in OPTICAL convention (z forward,
          x right, y down). This rpy makes the link an optical frame so optical-z
-         maps to base_link +x (forward). -->
-    <origin xyz="0.45 0.24 0.65" rpy="-1.5708 0.0 -1.5708"/>
+         maps to base_link +x (forward).
+         Height measured on hardware: lens ~0.45 m above the ground (base_link
+         origin is at ground level: wheel center z=0.16 - wheel_radius 0.16 = 0).
+         The old 0.65 was 20 cm too high and pushed floor/wall points below z=0. -->
+    <origin xyz="0.45 0.24 0.45" rpy="-1.5708 0.0 -1.5708"/>
   </joint>
   <link name="xtm60_right_link">
@@ -107,5 +110,10 @@
     <parent link="base_link"/>
     <child link="xtm60_right_link"/>
-    <!-- optical frame: z forward -> base_link +x (see left joint note) -->
+    <!-- optical frame: z forward -> base_link +x (see left joint note).
+         RIGHT radar was relocated out of the box onto the right armrest, taped,
+         ~20 cm higher than the original mount -> ~0.65 m above ground. The
+         lateral/forward offset on the armrest is approximate and MUST be
+         re-measured / calibrated in RViz against the left cloud before relying
+         on the merged map. Placeholder below. -->
     <origin xyz="0.45 -0.24 0.65" rpy="-1.5708 0.0 -1.5708"/>
   </joint>

Commit message: feat(ekf-pose-mapping): 实现单雷达纯EKF位姿建图链路并完成审查修复
关闭RTAB-Map所有几何配准，以EKF输出作为唯一位姿源建图，避免窄视场雷达的ICP滑移失真
修复D034/D168：融合节点使用源帧采集时间戳而非发布墙钟作为输出点云时间戳
修复D178：融合节点按点云采集时间戳查询TF，不可用时跳过该帧而非使用最新TF
修复D179：显式剔除点云中的(0,0,0)占位点与非有限值点
新增地平面自动标定节点，自动计算雷达高度与俯仰并发布TF
统一左右XT-M60雷达的设备端成像参数配置
调整URDF移除左雷达固定joint，由标定节点独占TF所有权
修正EKF配置中轮速yaw融合逻辑
更新单雷达建图启动脚本与RViz配置
新增相关单元测试与项目文档

File: src/wheelchair_description/urdf/wheelchair.urdf.xacro (robot description, xacro)
@@ -78,24 +78,17 @@
     <origin xyz="0.45 0.0 0.65" rpy="0.0 -0.0873 0.0"/>
   </joint>
-  <link name="xtm60_left_link">
-    <visual>
-      <origin xyz="0 0 0" rpy="0 0 0"/>
-      <geometry>
-        <box size="0.10 0.06 0.04"/>
-      </geometry>
-      <material name="laser_red"/>
-    </visual>
-  </link>
-  <joint name="xtm60_left_fixed_joint" type="fixed">
-    <parent link="base_link"/>
-    <child link="xtm60_left_link"/>
-    <!-- XT-M60 (ToF camera) publishes points in OPTICAL convention (z forward,
-         x right, y down). This rpy makes the link an optical frame so optical-z
-         maps to base_link +x (forward).
-         Height measured on hardware: lens ~0.45 m above the ground (base_link
-         origin is at ground level: wheel center z=0.16 - wheel_radius 0.16 = 0).
-         The old 0.65 was 20 cm too high and pushed floor/wall points below z=0. -->
-    <origin xyz="0.45 0.24 0.45" rpy="-1.5708 0.0 -1.5708"/>
-  </joint>
+  <!-- ============================================================
+       xtm60_left_link: TF edge base_link→xtm60_left_link is now OWNED by
+       ground_plane_calibrator_node (StaticTransformBroadcaster), which
+       calibrates the radar height (z) and pitch from the ground plane at
+       runtime (see .kiro/specs/ekf-pose-mapping, design 方案 A, req 2.4/2.7).
+       The former fixed joint (xyz=[0.45,0.24,0.45] rpy=[1.5708,0,1.5708],
+       z=0.45 placeholder) is removed here to avoid double-publishing the
+       same TF edge.  The calibrator reproduces the verified sensor
+       convention (z fwd, y up, x left) as R_CONV and adds calibrated pitch.
+       The xtm60_left_link visual box is dropped with the joint to keep the
+       URDF tree fully connected (the frame still exists via the calibrator's
+       TF broadcast). DO NOT re-add a fixed joint for this edge.
+       ============================================================ -->
   <link name="xtm60_right_link">
     <visual>
@@ -110,11 +103,12 @@
     <parent link="base_link"/>
     <child link="xtm60_right_link"/>
-    <!-- optical frame: z forward -> base_link +x (see left joint note).
-         RIGHT radar was relocated out of the box onto the right armrest, taped,
+    <!-- Same VERIFIED XT-M60 convention as the left radar: z fwd, y up, x left.
+         rpy=(pi/2,0,pi/2) (was -pi/2,0,-pi/2 which rolled the cloud 180 deg).
+         RIGHT radar relocated out of the box onto the right armrest, taped,
          ~20 cm higher than the original mount -> ~0.65 m above ground. The
          lateral/forward offset on the armrest is approximate and MUST be
          re-measured / calibrated in RViz against the left cloud before relying
          on the merged map. Placeholder below. -->
-    <origin xyz="0.45 -0.24 0.65" rpy="-1.5708 0.0 -1.5708"/>
+    <origin xyz="0.45 -0.24 0.65" rpy="1.5708 0.0 1.5708"/>
   </joint>
   <link name="imu_link">

Commit message: feat(manual_mapping): 添加多雷达选择支持，完善双雷达建图与遥测功能
- 新增双雷达扫描合并配置文件`scan_merger_dual.yaml`，适配单/双雷达扫描融合场景
- 重构launch文件与启动脚本，将原有`enable_xtm60_right`参数替换为统一的`radar`参数，支持left/right/both三种雷达模式
- 调整3D点云融合配置：将测距上限从12m提升至15m，放宽高度裁剪范围，关闭体素下采样以保留完整点云细节
- 修改RViz配置文件，将点云衰减时间改为99999，避免建图时点云过快消失影响观察
- 移除右雷达URDF中的固定关节与可视化模型，改为通过地面校准节点动态发布TF，支持自动校准雷达安装高度与俯仰角
- 更新`amp_view`启动脚本，适配双雷达的临时TF发布以保证点云可视化正常
- 更新所有相关脚本的注释与使用示例，补充右雷达与双雷达的启动方式

File: src/wheelchair_description/urdf/wheelchair.urdf.xacro (robot description, xacro)
@@ -91,25 +91,17 @@
        TF broadcast). DO NOT re-add a fixed joint for this edge.
        ============================================================ -->
-  <link name="xtm60_right_link">
-    <visual>
-      <origin xyz="0 0 0" rpy="0 0 0"/>
-      <geometry>
-        <box size="0.10 0.06 0.04"/>
-      </geometry>
-      <material name="laser_red"/>
-    </visual>
-  </link>
-  <joint name="xtm60_right_fixed_joint" type="fixed">
-    <parent link="base_link"/>
-    <child link="xtm60_right_link"/>
-    <!-- Same VERIFIED XT-M60 convention as the left radar: z fwd, y up, x left.
-         rpy=(pi/2,0,pi/2) (was -pi/2,0,-pi/2 which rolled the cloud 180 deg).
-         RIGHT radar relocated out of the box onto the right armrest, taped,
-         ~20 cm higher than the original mount -> ~0.65 m above ground. The
-         lateral/forward offset on the armrest is approximate and MUST be
-         re-measured / calibrated in RViz against the left cloud before relying
-         on the merged map. Placeholder below. -->
-    <origin xyz="0.45 -0.24 0.65" rpy="1.5708 0.0 1.5708"/>
-  </joint>
+  <!-- ============================================================
+       xtm60_right_link: TF edge base_link→xtm60_right_link is now OWNED by
+       ground_plane_calibrator_node (StaticTransformBroadcaster), same design
+       方案 A as the left radar. The calibrator auto-derives the right radar
+       height (z) and pitch from the ground plane (RANSAC on the first frames),
+       so the radar can be moved / re-aimed without editing this URDF. The
+       calibrator reproduces the verified sensor convention (z fwd, y up,
+       x left) as R_CONV and adds the calibrated pitch. The link visual box is
+       dropped with the joint to keep the URDF tree fully connected (the frame
+       still exists via the calibrator's TF broadcast). DO NOT re-add a fixed
+       joint for this edge. amp_view (which does NOT run the calibrator)
+       publishes a nominal static TF for this edge itself.
+       ============================================================ -->
   <link name="imu_link">
     <visual>
