Commit message: docs(hardware,mapping): add comprehensive acceptance and diagnostic documentation
- Add project handoff and memory documents for context preservation
- Add hardware audit, acceptance reports, and diagnostic documentation
* Camera array and FD07 array reports with diagnostics
* H30 IMU bringup and installation measurements
* XT M60 dual/single lidar bringup with interference mitigation and recovery
* Pointcloud amplitude analysis and orientation reports
* ZLAC encoder readonly configuration report
* Vendor configuration exports as binary evidence (192.168.0.101, 192.168.1.101, xintan_windows)
- Add mapping acceptance documentation for right lidar stage 1 validation
- Add 50+ diagnostic and validation scripts for hardware subsystems
* Camera array and ROS diagnostics
* FD07 array diagnostics and ROS integration
* H30 static IMU diagnostics
* XT M60 signal, cloud, orientation, phase, and resource diagnostics
* XT M60 configuration management and readonly feedback diagnostics
* UDP shutdown and quality gate soak testing
- Add mapping control scripts for right lidar stage 1 mapping workflow
- Update sensor adapter nodes with enhanced error handling and configuration
- Update RViz configuration and operator workbench panels for hardware visualization
- Add mapping manager quality gate and accumulator test coverage
- Add launch configurations for right lidar stage 1 mapping and stage 1 mapping contracts
- Add RViz hardware and XT M60 workbench configurations
- Normalize .gitignore with comprehensive sections and add .gitattributes for vendor evidence
- Preserve vendor exports as binary artifacts for acceptance evidence traceability

File: src/wheelchair_description/urdf/wheelchair.urdf.xacro (robot description, xacro)
@@ -78,30 +78,39 @@
     <origin xyz="0.45 0.0 0.65" rpy="0.0 -0.0873 0.0"/>
   </joint>
-  <!-- ============================================================
-       xtm60_left_link: TF edge base_link→xtm60_left_link is now OWNED by
-       ground_plane_calibrator_node (StaticTransformBroadcaster), which
-       calibrates the radar height (z) and pitch from the ground plane at
-       runtime (see .kiro/specs/ekf-pose-mapping, design 方案 A, req 2.4/2.7).
-       The former fixed joint (xyz=[0.45,0.24,0.45] rpy=[1.5708,0,1.5708],
-       z=0.45 placeholder) is removed here to avoid double-publishing the
-       same TF edge.  The calibrator reproduces the verified sensor
-       convention (z fwd, y up, x left) as R_CONV and adds calibrated pitch.
-       The xtm60_left_link visual box is dropped with the joint to keep the
-       URDF tree fully connected (the frame still exists via the calibrator's
-       TF broadcast). DO NOT re-add a fixed joint for this edge.
-       ============================================================ -->
-  <!-- ============================================================
-       xtm60_right_link: TF edge base_link→xtm60_right_link is now OWNED by
-       ground_plane_calibrator_node (StaticTransformBroadcaster), same design
-       方案 A as the left radar. The calibrator auto-derives the right radar
-       height (z) and pitch from the ground plane (RANSAC on the first frames),
-       so the radar can be moved / re-aimed without editing this URDF. The
-       calibrator reproduces the verified sensor convention (z fwd, y up,
-       x left) as R_CONV and adds the calibrated pitch. The link visual box is
-       dropped with the joint to keep the URDF tree fully connected (the frame
-       still exists via the calibrator's TF broadcast). DO NOT re-add a fixed
-       joint for this edge. amp_view (which does NOT run the calibrator)
-       publishes a nominal static TF for this edge itself.
-       ============================================================ -->
+  <!-- XT-M60 SDK coordinates are +z forward, +x left and +y up. The historical
+       ground_plane_calibrator source/executable is absent from this branch, so
+       robot_state_publisher is the single TF owner again. Lateral separation
+       (~0.60 m) and optical-centre height (0.735 m) are user measurements;
+       x=0.45 m remains the previous unverified longitudinal estimate. -->
+  <xacro:macro name="xtm60_link" params="name xyz rpy">
+    <link name="${name}">
+      <visual>
+        <origin xyz="0 0 0" rpy="0 0 0"/>
+        <geometry>
+          <box size="0.037 0.075 0.055"/>
+        </geometry>
+        <material name="laser_red"/>
+      </visual>
+    </link>
+    <joint name="${name}_fixed_joint" type="fixed">
+      <parent link="base_link"/>
+      <child link="${name}"/>
+      <origin xyz="${xyz}" rpy="${rpy}"/>
+    </joint>
+  </xacro:macro>
+  <!-- Left roll/pitch retains the last reliable floor-visible calibration from
+       feature/fastlio-narrow-fov-mapping (45b1163); current left floor fitting
+       selected a non-floor surface, so it was not used to overwrite this. -->
+  <xacro:xtm60_link
+    name="xtm60_left_link"
+    xyz="0.45 0.30 0.735"
+    rpy="1.5515153364 -0.0136154207 1.5709313394"/>
+  <!-- Right roll/pitch comes from the 2026-07-24 30-frame ground-plane repeat.
+       Horizontal yaw is constrained to optical-forward = base +x, not measured;
+       final dual-LiDAR yaw/xyz calibration remains required before fusion. -->
+  <xacro:xtm60_link
+    name="xtm60_right_link"
+    xyz="0.45 -0.30 0.735"
+    rpy="1.7071165220 0.0265268546 1.5744345976"/>
   <link name="imu_link">
     <visual>
@@ -118,5 +127,7 @@
     <parent link="base_link"/>
     <child link="imu_link"/>
-    <origin xyz="0.0 0.0 0.45" rpy="0.0 0.0 0.0"/>
+    <!-- Roll/pitch from the 2026-07-22 user-confirmed level 60 s gravity
+         capture. Yaw and xyz remain uncalibrated estimates. -->
+    <origin xyz="0.0 0.0 0.45" rpy="0.0098981264 0.0011002597 0.0"/>
   </joint>
   <xacro:macro name="camera_link" params="name xyz rpy">

Commit message: backup: snapshot wheel-IMU mapping and cleanup state

File: src/wheelchair_description/urdf/wheelchair.urdf.xacro (robot description, xacro)
@@ -19,4 +19,10 @@
        default robot model must not publish this provisional TF. -->
   <xacro:arg name="include_blocked_right_lidar_for_mock" default="false"/>
+  <!-- Explicit real-data diagnostic opt-in; never makes the formal contract
+       APPROVED. Both radar translations come from one measured-layout profile.
+       The existing mock-only fixture remains unchanged for synthetic tests. -->
+  <xacro:arg name="diagnostic_measured_layout" default="false"/>
+  <xacro:arg name="diagnostic_layout_profile" default="$(find wheelchair_description)/config/diagnostic_measured_layout.yaml"/>
+  <xacro:property name="diag_layout" value="${xacro.load_yaml('$(arg diagnostic_layout_profile)')}"/>
   <link name="base_link">
     <visual>
@@ -106,9 +112,10 @@
        feature/fastlio-narrow-fov-mapping (45b1163); current left floor fitting
        selected a non-floor surface, so it was not used to overwrite this. -->
-  <xacro:xtm60_link
-    name="xtm60_left_link"
-    xyz="0.45 0.30 0.735"
-    rpy="1.5515153364 -0.0136154207 1.5709313394"/>
-  <xacro:if value="$(arg include_blocked_right_lidar_for_mock)">
+  <xacro:unless value="$(arg diagnostic_measured_layout)">
+    <xacro:xtm60_link
+      name="xtm60_left_link"
+      xyz="0.45 0.30 0.735"
+      rpy="1.5515153364 -0.0136154207 1.5709313394"/>
+    <xacro:if value="$(arg include_blocked_right_lidar_for_mock)">
     <!-- MOCK-ONLY historical candidate. It is not runtime-eligible for real
          hardware: longitudinal x/yaw are uncalibrated and the strict contract
@@ -119,4 +126,13 @@
       xyz="0.606 -0.24 0.499"
       rpy="1.5806995918 0.1564194958 1.5715764604"/>
+    </xacro:if>
+  </xacro:unless>
+  <xacro:if value="$(arg diagnostic_measured_layout)">
+    <xacro:xtm60_link name="xtm60_left_link"
+      xyz="${' '.join(map(str, diag_layout['sensors']['left']['xyz']))}"
+      rpy="${' '.join(map(str, diag_layout['sensors']['left']['rpy']))}"/>
+    <xacro:xtm60_link name="xtm60_right_link"
+      xyz="${' '.join(map(str, diag_layout['sensors']['right']['xyz']))}"
+      rpy="${' '.join(map(str, diag_layout['sensors']['right']['rpy']))}"/>
   </xacro:if>
   <link name="imu_link">
@@ -136,5 +152,11 @@
     <!-- Roll/pitch from the 2026-07-22 user-confirmed level 60 s gravity
          capture. Yaw and xyz remain uncalibrated estimates. -->
-    <origin xyz="0.0 0.0 0.45" rpy="0.0098981264 0.0011002597 0.0"/>
+    <xacro:unless value="$(arg diagnostic_measured_layout)">
+      <origin xyz="0.0 0.0 0.45" rpy="0.0098981264 0.0011002597 0.0"/>
+    </xacro:unless>
+    <xacro:if value="$(arg diagnostic_measured_layout)">
+      <origin xyz="${' '.join(map(str, diag_layout['sensors']['imu']['xyz']))}"
+        rpy="${' '.join(map(str, diag_layout['sensors']['imu']['rpy']))}"/>
+    </xacro:if>
   </joint>
   <xacro:macro name="camera_link" params="name xyz rpy">
